Commit message: updated model, removed old sim files

File: arm_description/model/temp/arm.urdf (robot description, URDF)
Before this commit: robot arm, 6 links, 5 joints
Links:
- added link ee, mass 0.027464; collision mesh filename=package://arm_description/model/meshes/ee.STL; visual mesh filename=package://arm_description/model/meshes/ee.STL
- link base_link: mass 0.436656281721509 -> 0.43666
- link link1: mass 0.356326079956351 -> 0.35633
- link link2: mass 0.267463974995638 -> 0.26746
- link link3: mass 0.222311320377135 -> 0.222311320377134
Joints:
- added joint J6: type continuous, parent link5, child ee, origin xyz=-0.0199666324199864 -0.0127552190119366 0.00382596102472059 rpy=-1.41021344284507 -0.0773897000977449 2.12675451737731, axis 0 0 1
- joint J1: limit (none) -> lower=-3.1415 upper=3.1415 effort=1 velocity=10; origin xyz=0 0 0.054376 rpy=1.5708 0 -0.17957 -> xyz=0.087103 -0.077154 0.054376 rpy=1.5708 0 -0.17957; type continuous -> revolute
- joint J2: axis 0.1786 0 0.98392 -> 0.178603115585449 0 0.983921199641095; origin xyz=-0.038353 0.0583 -0.0013209 rpy=0.011484 -0.0003636 0.063304 -> xyz=-0.0383525749921799 0.0583000000000001 -0.0013208705506468 rpy=0.0114835938093404 -0.000363602890144003 0.0633037833578822
- joint J3: axis 0.1786 0 0.98392 -> 0.178603115585449 0 0.983921199641095; origin xyz=0.010122 0.15967 -0.0018373 rpy=-0.034158 -0.0032425 -0.18927 -> xyz=0.01012184118035 0.159668946677294 -0.00183733450496954 rpy=-0.0341579908525323 -0.00324248866976051 -0.189267104095329
- joint J4: axis 0.97586 0.12771 -0.17714 -> 0.97586466350816 0.127708020083281 -0.17714067890384; origin xyz=-3.6363E-05 0.014877 0.010525 rpy=0.019243 0.0025524 -0.0034694 -> xyz=-3.63625649351731E-05 0.0148771771133325 0.0105252497783941 rpy=0.0192434154802188 0.00255235780533698 -0.00346944801670467
- joint J5: axis 0.17609 0.019561 0.98418 -> 0.176090142676508 0.0195610841602276 0.98417967142115; origin xyz=-0.13556 -0.017639 0.024605 rpy=-3.0186 0.32455 0.71945 -> xyz=-0.135560517031385 -0.0176394821004389 0.0246051802150107 rpy=-3.01860336767631 0.324554663782284 0.719451490827395

File: arm_description/model/temp/robot_arm/urdf/robot_arm.urdf (robot description, URDF)
Before this commit: robot arm, 6 links, 5 joints
Links:
- link base_link: geometry collision mesh filename=package://robot_arm/meshes/base_link.STL; visual mesh filename=package://robot_arm/meshes/base_link.STL
- link link1: geometry collision mesh filename=package://robot_arm/meshes/link1.STL; visual mesh filename=package://robot_arm/meshes/link1.STL
- link link2: geometry collision mesh filename=package://robot_arm/meshes/link2.STL; visual mesh filename=package://robot_arm/meshes/link2.STL
- link link3: geometry collision mesh filename=package://robot_arm/meshes/link3.STL; visual mesh filename=package://robot_arm/meshes/link3.STL
- link link4: geometry collision mesh filename=package://robot_arm/meshes/link4.STL; visual mesh filename=package://robot_arm/meshes/link4.STL
- link link5: geometry collision mesh filename=package://robot_arm/meshes/link5.STL; visual mesh filename=package://robot_arm/meshes/link5.STL
